Commit message: Added some more walls to show where texture is projecting, but still don't have working image.

File: projector_test/urdf/projector_test.xacro (robot description, xacro)
@@ -18,4 +18,36 @@
   <child link="link_wall1" />
 </joint>
+<link name="link_wall2">
+  <visual>
+    <geometry>
+      <box size="10 10 0.1" />
+    </geometry>
+  </visual>
+  <inertial>
+    <mass value="1.0"/>
+    <inertia ixx="1.0" ixy="0.0" ixz="0.0" iyy="1.0" iyz="0.0" izz="1.0" />
+  </inertial>
+</link>
+<joint name="joint_wall2" type="fixed">
+  <origin xyz="0 0 10.0" rpy="0 0 0" />
+  <parent link="world" />
+  <child link="link_wall2" />
+</joint>
+<link name="link_wall3">
+  <visual>
+    <geometry>
+      <box size="10.0 0.1 20.0" />
+    </geometry>
+  </visual>
+  <inertial>
+    <mass value="1.0"/>
+    <inertia ixx="1.0" ixy="0.0" ixz="0.0" iyy="1.0" iyz="0.0" izz="1.0" />
+  </inertial>
+</link>
+<joint name="joint_wall3" type="fixed">
+  <origin xyz="0 5.0 0.0" rpy="0 0 0" />
+  <parent link="world" />
+  <child link="link_wall3" />
+</joint>
 <link name="link_projector">
   <visual>
@@ -30,12 +62,15 @@
 </link>
 <joint name="joint_projector" type="fixed">
-  <origin xyz="0 0 2.0" rpy="0 0 0" />
+  <origin xyz="0 0 2.0" rpy="0.0 0 0" />
   <parent link="world" />
   <child link="link_projector" />
 </joint>
 <gazebo reference="link_projector">
-  <projector name="projector_test">
+  <!--sensor type="projector" name="projector_tester"-->
+  <projector name="projector_test1">
     <pose>0 0 0 0 0 0</pose>
+    <!-- this isn't getting loaded properly -->
     <texture>$(find projector_test)/urdf/test_pattern.png</texture>
+    <!--texture>test_pattern.png</texture-->
     <fov>0.6</fov>
     <near_clip>0.1</near_clip>
@@ -43,3 +78,18 @@
   </projector>
 </gazebo>
+<gazebo if="false">
+  <!-- Not sure if this is necessary, didn't need it elsewhere though some
+      projector things were screwy -->
+    <plugin name="projector_test_controller" filename="libgazebo_ros_projector.so">
+      <projector>projector_test1</projector>
+      <alwaysOn>true</alwaysOn>
+      <updateRate>5.0</updateRate>
+      <textureName>$(find projector_test/urdf/test_pattern.png</textureName>
+      <!-- what is the filter for? -->
+      <filterTextureName>$(find projector_test)/urdf/test_pattern.png</filterTextureName>
+      <textureTopicName>projector_test/image</textureTopicName>
+      <projectorTopicName>projector_test/projector</projectorTopicName>
+    </plugin>
+    <!--/sensor-->
+  </gazebo>
 </robot>

Commit message: Still can't get the texture to load, but using a system installed texture works, also setting pose of joint works okay.

File: projector_test/urdf/projector_test.xacro (robot description, xacro)
@@ -62,5 +62,5 @@
 </link>
 <joint name="joint_projector" type="fixed">
-  <origin xyz="0 0 2.0" rpy="0.0 0 0" />
+  <origin xyz="0 0 2.0" rpy="-0.77 0 0" />
   <parent link="world" />
   <child link="link_projector" />
@@ -71,7 +71,9 @@
     <pose>0 0 0 0 0 0</pose>
     <!-- this isn't getting loaded properly -->
-    <texture>$(find projector_test)/urdf/test_pattern.png</texture>
+    <!--texture>$(find projector_test)/urdf/test_pattern.png</texture-->
+    <!-- this doesn't work even with setting GAZEBO_RESOURCE_PATH -->
     <!--texture>test_pattern.png</texture-->
-    <fov>0.6</fov>
+    <texture>stereo_projection_pattern_high_res_red.png</texture>
+    <fov>0.95</fov>
     <near_clip>0.1</near_clip>
     <far_clip>10.0</far_clip>

Commit message: Confirm that setting the projector pose produces glitchy output as it does in sdf http://answers.gazebosim.org/question/5223/setting-projector-pose-vs-enclosing-link-pose/

File: projector_test/urdf/projector_test.xacro (robot description, xacro)
@@ -62,5 +62,5 @@
 </link>
 <joint name="joint_projector" type="fixed">
-  <origin xyz="0 0 2.0" rpy="-0.77 0 0" />
+  <origin xyz="0 0 2.0" rpy="-0.0 0 0" />
   <parent link="world" />
   <child link="link_projector" />
@@ -69,5 +69,5 @@
   <!--sensor type="projector" name="projector_tester"-->
   <projector name="projector_test1">
-    <pose>0 0 0 0 0 0</pose>
+    <pose>0 0 0 -0.88 0 0</pose>
     <!-- this isn't getting loaded properly -->
     <!--texture>$(find projector_test)/urdf/test_pattern.png</texture-->
