Commit message: Successfully creating a segmented hierarch, next make a robot_state_publisher and check in rviz.
This works now:

rosrun xacro xacro.py testbot.xacro > model.urdf
rosrun urdfdom check_urdf model.urdf
rosrun urdfdom urdf_to_graphiz model.urdf
evince testbot.pdf

File: testbot_description/urdf/testbot.xacro (robot description, xacro)
@@ -1,23 +1,23 @@
 <?xml version="1.0"?>
-<robot name="testbot" xmlns:xacro="https://github.com/lucasw/testbot">
+<robot name="testbot" xmlns:xacro="http://www.ros.org/wiki/xacro">
 <!-- http://answers.ros.org/question/38956/pass-parameters-to-xacro-in-launch-file/ -->
 <xacro:property name="seg_length" value="0.2" />
 <xacro:property name="seg_width" value="0.15" />
 <xacro:property name="seg_height" value="0.1" />
-<link name="base_link" />
-<xacro:macro name="segment" params="parent post_fix length width height" />
+<xacro:macro name="segment" params="parent postfix length width height">
   <link name="link_${postfix}">
-    <collision>
+<!--    <collision>
       <origin xyz="0 0 0" rpy="0 0 0" />
       <geometry>
         <box size="${length} ${width} ${height}" />
       </geometry>
-      <visual>
+    </collision>
+    <visual>
         <origin xyz="0 0 0" rpy="0 0 0" />
         <geometry>
           <box size="${length} ${width} ${height}" />
         </geometry>
-      </visual>
-      <inertial>
+    </visual>
+    <inertial>
         <origin xyz="0 0 0" rpy="0 0 0" />
         <mass value="1.0" />
@@ -26,11 +26,23 @@
           iyy="1.0" iyz="0.0"
           izz="1.0" />
-      </inertial>
-      <joint name="joint_${postfix}" type="revolute">
+    </inertial>
+    -->
+  </link>
+  <joint name="joint_${postfix}" type="revolute">
         <parent link="${parent}" />
-        <child link="link_${parent}" />
-      </joint>
-    </collision>
-  </link>
+        <child link="link_${postfix}" />
+        <origin xyz="${length/2 + 0.05} 0 0" rpy="0 0 0" />
+        <axis xyz="0 0 1" />
+        <limit effort="1000.0" lower="-0.5" upper="0.5" velocity="0.5" />
+  </joint>
 </xacro:macro>
+<link name="base_link" />
+<xacro:segment parent="base_link" postfix="1" length="${seg_length}" width="${seg_width}" height="${seg_height}" />
+     <xacro:segment parent="link_1" postfix="2" length="${seg_length}" width="${seg_width}" height="${seg_height}" />
+<xacro:segment parent="link_2" postfix="3" length="${seg_length}" width="${seg_width}" height="${seg_height}" />
+<xacro:segment parent="link_3" postfix="4" length="${seg_length}" width="${seg_width}" height="${seg_height}" />
+<!--
+<xacro:segment parent="link_4" postfix="5" length="${seg_length}" width="${seg_width}" height="${seg_height}" />
+<xacro:segment parent="link_5" postfix="6" length="${seg_length}" width="${seg_width}" height="${seg_height}" />
+-->
 </robot>

Commit message: Have the visual working by using the RobotModel rviz plugin, some of the tutorials take that for granted.

File: testbot_description/urdf/testbot.xacro (robot description, xacro)
@@ -7,5 +7,15 @@
 <xacro:macro name="segment" params="parent postfix length width height">
   <link name="link_${postfix}">
-<!--    <collision>
+    <visual>
+        <origin xyz="0 0 0" rpy="0 0 0" />
+        <geometry>
+          <box size="${length} ${width} ${height}" />
+        </geometry>
+        <material name="grey_${postfix}">
+          <color rgba="0.5 0.5 0.5 1" />
+        </material>
+    </visual>
+    <!--
+    <collision>
       <origin xyz="0 0 0" rpy="0 0 0" />
       <geometry>
@@ -13,10 +23,4 @@
       </geometry>
     </collision>
-    <visual>
-        <origin xyz="0 0 0" rpy="0 0 0" />
-        <geometry>
-          <box size="${length} ${width} ${height}" />
-        </geometry>
-    </visual>
     <inertial>
         <origin xyz="0 0 0" rpy="0 0 0" />
@@ -33,4 +37,5 @@
         <child link="link_${postfix}" />
         <origin xyz="${length/2 + 0.05} 0 0" rpy="0 0 0" />
+        <!--pose xyz="${-length/2 - 0.05} 0 0" rpy="0 0 0" /-->
         <axis xyz="0 0 1" />
         <limit effort="1000.0" lower="-0.5" upper="0.5" velocity="0.5" />

Commit message: Adjust joint positions and visual positions so everything makes sense- so could use a dae at this point so the boxes aren't self-intersecting, but it isn't that important.  Next add some wheels.

File: testbot_description/urdf/testbot.xacro (robot description, xacro)
@@ -8,5 +8,5 @@
   <link name="link_${postfix}">
     <visual>
-        <origin xyz="0 0 0" rpy="0 0 0" />
+        <origin xyz="${length/2} 0 0" rpy="0 0 0" />
         <geometry>
           <box size="${length} ${width} ${height}" />
@@ -16,7 +16,6 @@
         </material>
     </visual>
-    <!--
     <collision>
-      <origin xyz="0 0 0" rpy="0 0 0" />
+      <origin xyz="${length/2} 0 0" rpy="0 0 0" />
       <geometry>
         <box size="${length} ${width} ${height}" />
@@ -24,5 +23,5 @@
     </collision>
     <inertial>
-        <origin xyz="0 0 0" rpy="0 0 0" />
+        <origin xyz="${length/2} 0 0" rpy="0 0 0" />
         <mass value="1.0" />
         <inertia
@@ -31,11 +30,9 @@
           izz="1.0" />
     </inertial>
-    -->
   </link>
   <joint name="joint_${postfix}" type="revolute">
         <parent link="${parent}" />
         <child link="link_${postfix}" />
-        <origin xyz="${length/2 + 0.05} 0 0" rpy="0 0 0" />
-        <!--pose xyz="${-length/2 - 0.05} 0 0" rpy="0 0 0" /-->
+        <origin xyz="${length} 0 0" rpy="0 0 0" />
         <axis xyz="0 0 1" />
         <limit effort="1000.0" lower="-0.5" upper="0.5" velocity="0.5" />

Commit message: This loads and scales the cube correctly.  The next step is to add a vertical cylinder to the cube in blender that will stand in for the joint.

File: testbot_description/urdf/testbot.xacro (robot description, xacro)
@@ -10,5 +10,6 @@
         <origin xyz="${length/2} 0 0" rpy="0 0 0" />
         <geometry>
-          <box size="${length} ${width} ${height}" />
+          <!--box size="${length} ${width} ${height}" /-->
+          <mesh filename="package://testbot_description/meshes/cube.dae" scale="${length/2} ${width/2} ${height/2}" />
         </geometry>
         <material name="grey_${postfix}">

Commit message: The purely visual rotation joints are in the correct places and look good, I'll want to make sure gazebo ignores them except as collision volumes when I get to gazebo integration.  The other thing to do is make the segments thicker but shorter and the rotational joints smaller, since I want to put wheels on the segments.

File: testbot_description/urdf/testbot.xacro (robot description, xacro)
@@ -2,4 +2,5 @@
 <robot name="testbot" xmlns:xacro="http://www.ros.org/wiki/xacro">
 <!-- http://answers.ros.org/question/38956/pass-parameters-to-xacro-in-launch-file/ -->
+<xacro:property name="pi" value="3.1415926535897931" />
 <xacro:property name="seg_length" value="0.2" />
 <xacro:property name="seg_width" value="0.15" />
@@ -11,5 +12,5 @@
         <geometry>
           <!--box size="${length} ${width} ${height}" /-->
-          <mesh filename="package://testbot_description/meshes/cube.dae" scale="${length/2} ${width/2} ${height/2}" />
+          <mesh filename="package://testbot_description/meshes/cube.dae" scale="${length/2} ${width/4} ${height/4}" />
         </geometry>
         <material name="grey_${postfix}">
@@ -20,5 +21,5 @@
       <origin xyz="${length/2} 0 0" rpy="0 0 0" />
       <geometry>
-        <box size="${length} ${width} ${height}" />
+        <box size="${length/2} ${width/2} ${height/2}" />
       </geometry>
     </collision>
@@ -32,4 +33,39 @@
     </inertial>
   </link>
+  <!-- This link is just here to provide a visual for the joint -->
+  <link name="link_joint_${postfix}">
+    <visual>
+        <origin xyz="0 0 0" rpy="${pi/2} 0 0" />
+        <geometry>
+          <!--box size="${length} ${width} ${height}" /-->
+          <mesh filename="package://testbot_description/meshes/cylinder.dae" scale="${length/4} ${length/4} ${length/4}" />
+        </geometry>
+        <material name="grey_${postfix}">
+          <color rgba="0.5 0.5 0.5 1" />
+        </material>
+    </visual>
+    <!-- Do I need this? Wouldn't want thin things to fall between segments -->
+    <collision>
+      <origin xyz="0 0 0" rpy="0 0 0" />
+      <geometry>
+        <box size="${length/3} ${length/3} ${length/3}" />
+      </geometry>
+    </collision>
+    <!-- Do I need this? -->
+    <!--inertial>
+        <origin xyz="0 0 0" rpy="0 0 0" />
+        <mass value="1.0" />
+        <inertia
+          ixx="1.0" ixy="0.0" ixz="0.0"
+          iyy="1.0" iyz="0.0"
+          izz="1.0" />
+    </inertial-->
+  </link>
+  <joint name="joint_link_${postfix}" type="fixed">
+        <parent link="${parent}" />
+        <child link="link_joint_${postfix}" />
+        <origin xyz="${length} 0 0" rpy="0 0 0" />
+        <axis xyz="0 0 1" />
+  </joint>
   <joint name="joint_${postfix}" type="revolute">
         <parent link="${parent}" />

Commit message: Made the cylinders smaller and segment cuboids bigger.

File: testbot_description/urdf/testbot.xacro (robot description, xacro)
@@ -6,4 +6,5 @@
 <xacro:property name="seg_width" value="0.15" />
 <xacro:property name="seg_height" value="0.1" />
+<xacro:property name="cyl_div" value="4.0" />
 <xacro:macro name="segment" params="parent postfix length width height">
   <link name="link_${postfix}">
@@ -12,5 +13,5 @@
         <geometry>
           <!--box size="${length} ${width} ${height}" /-->
-          <mesh filename="package://testbot_description/meshes/cube.dae" scale="${length/2} ${width/4} ${height/4}" />
+          <mesh filename="package://testbot_description/meshes/cube.dae" scale="${length/3} ${width/2} ${height/2}" />
         </geometry>
         <material name="grey_${postfix}">
@@ -39,5 +40,5 @@
         <geometry>
           <!--box size="${length} ${width} ${height}" /-->
-          <mesh filename="package://testbot_description/meshes/cylinder.dae" scale="${length/4} ${length/4} ${length/4}" />
+          <mesh filename="package://testbot_description/meshes/cylinder.dae" scale="${length/cyl_div} ${0.5 * length/cyl_div} ${length/cyl_div}" />
         </geometry>
         <material name="grey_${postfix}">

Commit message: Have wheels on one side, next turn into macro and put another wheel on other side.  Also add an axle purely visual link- Some of the visual it makes sense to bake into the dae file, but if they are to be insensitive to scaling then they need to be broken- it would be convenient to be able to add a second visual tag and make composite objects.

File: testbot_description/urdf/testbot.xacro (robot description, xacro)
@@ -8,4 +8,5 @@
 <xacro:property name="cyl_div" value="4.0" />
 <xacro:macro name="segment" params="parent postfix length width height">
+  <!-- the segment -->
   <link name="link_${postfix}">
     <visual>
@@ -43,5 +44,5 @@
         </geometry>
         <material name="grey_${postfix}">
-          <color rgba="0.5 0.5 0.5 1" />
+          <color rgba="0.3 0.3 0.3 1" />
         </material>
     </visual>
@@ -76,4 +77,36 @@
         <limit effort="1000.0" lower="-0.5" upper="0.5" velocity="0.5" />
   </joint>
+  <!-- left wheel axle, put in macro -->
+  <joint name="joint_axle_${postfix}" type="continuous">
+        <parent link="link_${postfix}" />
+        <child link="link_wheel_${postfix}" />
+        <origin xyz="${length/2} ${length/1.8} ${-length/4}" rpy="0 0 0" />
+        <axis xyz="0 1 0" />
+        <limit effort="1000.0" velocity="0.5" />
+  </joint>
+  <!-- left wheel, put in macro -->
+  <link name="link_wheel_${postfix}">
+    <visual>
+        <origin xyz="0 0 0" rpy="0 0 0" />
+        <geometry>
+          <!--box size="${length} ${width} ${height}" /-->
+          <mesh filename="package://testbot_description/meshes/cylinder.dae" scale="${length/4} ${length/8} ${length/4}" />
+        </geometry>
+    </visual>
+    <collision>
+      <origin xyz="0 0 0" rpy="0 0 0" />
+      <geometry>
+        <box size="${length/4} ${length/8} ${length/4}" />
+      </geometry>
+    </collision>
+    <inertial>
+        <origin xyz="0 0 0" rpy="0 0 0" />
+        <mass value="0.5" />
+        <inertia
+          ixx="1.0" ixy="0.0" ixz="0.0"
+          iyy="1.0" iyz="0.0"
+          izz="1.0" />
+    </inertial>
+  </link>
 </xacro:macro>
 <link name="base_link" />

Commit message: Now have macro for wheels, and left and right wheels.  Next look at passing parameters in from launch file, and gazebo integration.

File: testbot_description/urdf/testbot.xacro (robot description, xacro)
@@ -7,4 +7,44 @@
 <xacro:property name="seg_height" value="0.1" />
 <xacro:property name="cyl_div" value="4.0" />
+<xacro:macro name="wheel" params="dir parent postfix length width height">
+<!-- the name doesn't actually do anything, was hoping maybe it would
+       allow multiple visuals within the same link -->
+  <link name="link_wheel_${postfix}">
+    <visual name="vis1_${postfix}">
+        <origin xyz="0 0 0" rpy="0 0 0" />
+        <geometry>
+          <mesh filename="package://testbot_description/meshes/cylinder.dae" scale="${length/4} ${length/8} ${length/4}" />
+        </geometry>
+    </visual>
+    <!--visual name="vis2_${postfix}">
+        <origin xyz="0 -${length} 0" rpy="0 0 0" />
+        <geometry>
+          <mesh filename="package://testbot_description/meshes/cylinder.dae" scale="${length/4} ${length/8} ${length/4}" />
+        </geometry>
+    </visual-->
+    <collision>
+      <origin xyz="0 0 0" rpy="0 0 0" />
+      <geometry>
+        <box size="${length/4} ${length/8} ${length/4}" />
+      </geometry>
+    </collision>
+    <inertial>
+        <origin xyz="0 0 0" rpy="0 0 0" />
+        <mass value="0.5" />
+        <inertia
+          ixx="1.0" ixy="0.0" ixz="0.0"
+          iyy="1.0" iyz="0.0"
+          izz="1.0" />
+    </inertial>
+  </link>
+  <!-- left wheel axle -->
+  <joint name="joint_axle_${postfix}" type="continuous">
+        <parent link="${parent}" />
+        <child link="link_wheel_${postfix}" />
+        <origin xyz="${length/2} ${dir * length/1.8} ${-length/4}" rpy="0 0 0" />
+        <axis xyz="0 1 0" />
+        <limit effort="1000.0" velocity="0.5" />
+  </joint>
+</xacro:macro>
 <xacro:macro name="segment" params="parent postfix length width height">
   <!-- the segment -->
@@ -64,4 +104,5 @@
     </inertial-->
   </link>
+  <!-- this is just for visual purpose -->
   <joint name="joint_link_${postfix}" type="fixed">
         <parent link="${parent}" />
@@ -70,4 +111,5 @@
         <axis xyz="0 0 1" />
   </joint>
+  <!-- this is a functional joint -->
   <joint name="joint_${postfix}" type="revolute">
         <parent link="${parent}" />
@@ -77,36 +119,7 @@
         <limit effort="1000.0" lower="-0.5" upper="0.5" velocity="0.5" />
   </joint>
-  <!-- left wheel axle, put in macro -->
-  <joint name="joint_axle_${postfix}" type="continuous">
-        <parent link="link_${postfix}" />
-        <child link="link_wheel_${postfix}" />
-        <origin xyz="${length/2} ${length/1.8} ${-length/4}" rpy="0 0 0" />
-        <axis xyz="0 1 0" />
-        <limit effort="1000.0" velocity="0.5" />
-  </joint>
   <!-- left wheel, put in macro -->
-  <link name="link_wheel_${postfix}">
-    <visual>
-        <origin xyz="0 0 0" rpy="0 0 0" />
-        <geometry>
-          <!--box size="${length} ${width} ${height}" /-->
-          <mesh filename="package://testbot_description/meshes/cylinder.dae" scale="${length/4} ${length/8} ${length/4}" />
-        </geometry>
-    </visual>
-    <collision>
-      <origin xyz="0 0 0" rpy="0 0 0" />
-      <geometry>
-        <box size="${length/4} ${length/8} ${length/4}" />
-      </geometry>
-    </collision>
-    <inertial>
-        <origin xyz="0 0 0" rpy="0 0 0" />
-        <mass value="0.5" />
-        <inertia
-          ixx="1.0" ixy="0.0" ixz="0.0"
-          iyy="1.0" iyz="0.0"
-          izz="1.0" />
-    </inertial>
-  </link>
+  <xacro:wheel parent="link_${postfix}" postfix="right_${postfix}" dir="1.0" length="${length}" width="${width}" height="${height}"  />
+  <xacro:wheel parent="link_${postfix}" postfix="left_${postfix}" dir="-1.0" length="${length}" width="${width}" height="${height}"  />
 </xacro:macro>
 <link name="base_link" />

Commit message: Adding untested gazebo transmission elements following the http://gazebosim.org/wiki/Tutorials/1.9/ROS_Control_with_Gazebo tutorial.

File: testbot_description/urdf/testbot.xacro (robot description, xacro)
@@ -26,10 +26,10 @@
       <origin xyz="0 0 0" rpy="0 0 0" />
       <geometry>
-        <box size="${length/4} ${length/8} ${length/4}" />
+        <cylinder length="${length/4}" radius="${length/4}" />
       </geometry>
     </collision>
     <inertial>
         <origin xyz="0 0 0" rpy="0 0 0" />
-        <mass value="0.5" />
+        <mass value="2" />
         <inertia
           ixx="1.0" ixy="0.0" ixz="0.0"
@@ -68,5 +68,5 @@
     <inertial>
         <origin xyz="${length/2} 0 0" rpy="0 0 0" />
-        <mass value="1.0" />
+        <mass value="20.0" />
         <inertia
           ixx="1.0" ixy="0.0" ixz="0.0"
@@ -75,4 +75,8 @@
     </inertial>
   </link>
+  <gazebo reference="link_${postfix}">
+    <mu1>0.2</mu1>
+    <mu2>0.2</mu2>
+  </gazebo>
   <!-- This link is just here to provide a visual for the joint -->
   <link name="link_joint_${postfix}">
@@ -91,5 +95,5 @@
       <origin xyz="0 0 0" rpy="0 0 0" />
       <geometry>
-        <box size="${length/3} ${length/3} ${length/3}" />
+        <cylinder length="${0.5 * length/cyl_div}" radius="${length/cyl_div" />
       </geometry>
     </collision>
@@ -111,5 +115,5 @@
         <axis xyz="0 0 1" />
   </joint>
-  <!-- this is a functional joint -->
+  <!-- this is a functional joint between segments -->
   <joint name="joint_${postfix}" type="revolute">
         <parent link="${parent}" />
@@ -118,9 +122,26 @@
         <axis xyz="0 0 1" />
         <limit effort="1000.0" lower="-0.5" upper="0.5" velocity="0.5" />
+        <dynamics damping="0.5" />
   </joint>
+  <transmission name="tran_joint_seg_${postfix}">
+    <type>transmission_interface/SimpleTransmission</type>
+    <joint name="joint_${postfix}" />
+    <actuator name="motor_seg_${postfix}">
+      <hardwareInterface>EffortJointInterface</hardwareInterface>
+      <mechanicalReduction>1</mechanicalReduction>
+    </actuator>
+  </transmission>
   <!-- left wheel, put in macro -->
   <xacro:wheel parent="link_${postfix}" postfix="right_${postfix}" dir="1.0" length="${length}" width="${width}" height="${height}"  />
   <xacro:wheel parent="link_${postfix}" postfix="left_${postfix}" dir="-1.0" length="${length}" width="${width}" height="${height}"  />
 </xacro:macro>
+<gazebo>
+  <plugin name="gazebo_ros_control" filename="libgazebo_ros_control.so">
+    <!-- will default to robot name -->
+    <!--robotNamespace>/testbot</robotNamespace-->
+    <!-- TBD rename this later -->
+    <robotParam>/robot_description</robotparam>
+  </plugin>
+</gazebo>
 <link name="base_link" />
 <xacro:segment parent="base_link" postfix="1" length="${seg_length}" width="${seg_width}" height="${seg_height}" />

Commit message: Fixed some bugs encountered when attempting to
roslaunch testbot_gazebo testbot_gazebo.launch

but still not working yet.  Current error is:

[ERROR] [1384774745.237610026, 0.406000000]: This robot has a joint named "joint_1" which is not in the gazebo model.
[FATAL] [1384774745.237833810, 0.406000000]: Could not initialize robot simulation interface

Also seeing this warning:

[ INFO] [1384774745.224143962, 0.406000000]: pluginlib WARNING: In file /tmp/buildd/ros-hydro-gazebo-ros-control-2.3.3-0raring-20131024-0611/src/default_robot_hw_sim.cpp PLUGINLIB_DECLARE_CLASS is deprecated, please use PLUGINLIB_EXPORT_CLASS instead. You can run the script 'plugin_macro_update' provided with pluginlib in your package source folder to automatically and recursively update legacy macros.  Base = base_class_type, Derived = derived_class_type

File: testbot_description/urdf/testbot.xacro (robot description, xacro)
@@ -80,5 +80,5 @@
   </gazebo>
   <!-- This link is just here to provide a visual for the joint -->
-  <link name="link_joint_${postfix}">
+  <link name="link_jointviz_${postfix}">
     <visual>
         <origin xyz="0 0 0" rpy="${pi/2} 0 0" />
@@ -95,5 +95,5 @@
       <origin xyz="0 0 0" rpy="0 0 0" />
       <geometry>
-        <cylinder length="${0.5 * length/cyl_div}" radius="${length/cyl_div" />
+        <cylinder length="${0.5 * length/cyl_div}" radius="${length/cyl_div}" />
       </geometry>
     </collision>
@@ -109,7 +109,7 @@
   </link>
   <!-- this is just for visual purpose -->
-  <joint name="joint_link_${postfix}" type="fixed">
+  <joint name="joint_linkviz_${postfix}" type="fixed">
         <parent link="${parent}" />
-        <child link="link_joint_${postfix}" />
+        <child link="link_jointviz_${postfix}" />
         <origin xyz="${length} 0 0" rpy="0 0 0" />
         <axis xyz="0 0 1" />

Commit message: Ifed out the unnecessary visual elements, but still getting the 'not in the gazebo model' error

File: testbot_description/urdf/testbot.xacro (robot description, xacro)
@@ -80,4 +80,5 @@
   </gazebo>
   <!-- This link is just here to provide a visual for the joint -->
+  <xacro:if value="false">
   <link name="link_jointviz_${postfix}">
     <visual>
@@ -115,6 +116,7 @@
         <axis xyz="0 0 1" />
   </joint>
+  </xacro:if>
   <!-- this is a functional joint between segments -->
-  <joint name="joint_${postfix}" type="revolute">
+  <joint name="joint_seg_${postfix}" type="revolute">
         <parent link="${parent}" />
         <child link="link_${postfix}" />
@@ -126,5 +128,5 @@
   <transmission name="tran_joint_seg_${postfix}">
     <type>transmission_interface/SimpleTransmission</type>
-    <joint name="joint_${postfix}" />
+    <joint name="joint_seg_${postfix}" />
     <actuator name="motor_seg_${postfix}">
       <hardwareInterface>EffortJointInterface</hardwareInterface>
@@ -132,7 +134,9 @@
     </actuator>
   </transmission>
-  <!-- left wheel, put in macro -->
+  <!-- wheels -->
+  <xacro:if value="false">
   <xacro:wheel parent="link_${postfix}" postfix="right_${postfix}" dir="1.0" length="${length}" width="${width}" height="${height}"  />
   <xacro:wheel parent="link_${postfix}" postfix="left_${postfix}" dir="-1.0" length="${length}" width="${width}" height="${height}"  />
+  </xacro:if>
 </xacro:macro>
 <gazebo>
