Commit message: I think the problem http://answers.ros.org/question/102276/this-robot-has-a-joint-named-foo-which-is-not-in-the-gazebo-model/ was due to having a gazebo controlled joint that attached to a link with no physical properties.  There are some other namespace adjustments that I've made that seemed also necessary, though I'm getting a 'Controller Spawner couldn't find the expected controller_manager ROS interface.' warning right now.  But the model appears in gazebo at least.

File: testbot_description/urdf/testbot.xacro (robot description, xacro)
@@ -145,9 +145,38 @@
     <robotNamespace>/testbot</robotNamespace>
     <!-- TBD rename this later -->
+    <!--robotParam>/robot_description</robotParam-->
     <robotParam>/testbot/robot_description</robotParam>
   </plugin>
 </gazebo>
-<link name="base_link" />
-<xacro:segment parent="base_link" postfix="1" length="${seg_length}" width="${seg_width}" height="${seg_height}" />
+<link name="base_link"/>
+<link name="head">
+    <visual>
+        <origin xyz="0 0 0" rpy="0 0 0" />
+        <geometry>
+          <mesh filename="package://testbot_description/meshes/cylinder.dae" scale="${seg_length/3} ${seg_length/6} ${seg_length/3}" />
+        </geometry>
+    </visual>
+    <collision>
+      <origin xyz="0 0 0" rpy="0 0 0" />
+      <geometry>
+        <cylinder length="${seg_length/6}" radius="${seg_length/3}" />
+      </geometry>
+    </collision>
+    <inertial>
+        <origin xyz="0 0 0" rpy="0 0 0" />
+        <mass value="1" />
+        <inertia
+          ixx="1.0" ixy="0.0" ixz="0.0"
+          iyy="1.0" iyz="0.0"
+          izz="1.0" />
+    </inertial>
+</link>
+  <joint name="joint_base_head" type="fixed">
+        <parent link="base_link" />
+        <child link="head" />
+        <origin xyz="0 0 0" rpy="0 0 0" />
+        <axis xyz="0 0 1" />
+  </joint>
+<xacro:segment parent="head" postfix="1" length="${seg_length}" width="${seg_width}" height="${seg_height}" />
 <xacro:segment parent="link_1" postfix="2" length="${seg_length}" width="${seg_width}" height="${seg_height}" />
 <xacro:segment parent="link_2" postfix="3" length="${seg_length}" width="${seg_width}" height="${seg_height}" />

Commit message: Made wheels work, need to rotate the dae file to restore that to working order.

File: testbot_description/urdf/testbot.xacro (robot description, xacro)
@@ -7,12 +7,19 @@
 <xacro:property name="seg_height" value="0.1" />
 <xacro:property name="cyl_div" value="4.0" />
+<!--
+    Wheel
+    =====
+ -->
 <xacro:macro name="wheel" params="dir parent postfix length width height">
 <!-- the name doesn't actually do anything, was hoping maybe it would
        allow multiple visuals within the same link -->
   <link name="link_wheel_${postfix}">
-    <visual name="vis1_${postfix}">
-        <origin xyz="0 0 0" rpy="0 0 0" />
-        <geometry>
-          <mesh filename="package://testbot_description/meshes/cylinder.dae" scale="${length/4} ${length/8} ${length/4}" />
+    <visual>
+      <!-- use this when using the cylinder primitive, the mesh doesn't align -->
+      <origin xyz="0 0 0" rpy="${pi/2} 0 0" />
+        <geometry>
+          <cylinder length="${length/4}" radius="${length/4}" />
+          <!-- TODO rotate the mesh so it aligns with the cylinder -->
+          <!--mesh filename="package://testbot_description/meshes/cylinder.dae" scale="${length/4} ${length/8} ${length/4}" /-->
         </geometry>
     </visual>
@@ -24,5 +31,5 @@
     </visual-->
     <collision>
-      <origin xyz="0 0 0" rpy="0 0 0" />
+      <origin xyz="0 0 0" rpy="${pi/2} 0 0" />
       <geometry>
         <cylinder length="${length/4}" radius="${length/4}" />
@@ -38,5 +45,5 @@
     </inertial>
   </link>
-  <!-- left wheel axle -->
+  <!-- wheel axle -->
   <joint name="joint_axle_${postfix}" type="continuous">
         <parent link="${parent}" />
@@ -47,4 +54,11 @@
   </joint>
 </xacro:macro>
+<!--
+  end wheel
+  -->
+<!--
+  Segment
+  =======
+-->
 <xacro:macro name="segment" params="parent postfix length width height">
   <!-- the segment -->
@@ -54,5 +68,6 @@
         <geometry>
           <!--box size="${length} ${width} ${height}" /-->
-          <mesh filename="package://testbot_description/meshes/cube.dae" scale="${length/3} ${width/2} ${height/2}" />
+          <mesh filename="package://testbot_description/meshes/cube.dae"
+              scale="${length/3} ${width/2} ${height/2}" />
         </geometry>
         <material name="grey_${postfix}">
@@ -135,9 +150,13 @@
   </transmission>
   <!-- wheels -->
-  <xacro:if value="false">
+  <xacro:if value="true">
   <xacro:wheel parent="link_${postfix}" postfix="right_${postfix}" dir="1.0" length="${length}" width="${width}" height="${height}"  />
   <xacro:wheel parent="link_${postfix}" postfix="left_${postfix}" dir="-1.0" length="${length}" width="${width}" height="${height}"  />
   </xacro:if>
 </xacro:macro>
+<!--
+  End segment section
+  ===================
+-->
 <gazebo>
   <plugin name="gazebo_ros_control" filename="libgazebo_ros_control.so">
@@ -153,17 +172,21 @@
 <link name="head">
     <visual>
-        <origin xyz="0 0 0" rpy="0 0 0" />
-        <geometry>
-          <mesh filename="package://testbot_description/meshes/cylinder.dae" scale="${seg_length/3} ${seg_length/6} ${seg_length/3}" />
-        </geometry>
-    </visual>
-    <collision>
-      <origin xyz="0 0 0" rpy="0 0 0" />
-      <geometry>
-        <cylinder length="${seg_length/6}" radius="${seg_length/3}" />
+        <origin xyz="${seg_length/2} 0 0" rpy="0 0 0" />
+        <geometry>
+          <mesh filename="package://testbot_description/meshes/cube.dae"
+              scale="${seg_length/3} ${seg_width/2} ${seg_height/2}" />
+          <!--mesh filename="package://testbot_description/meshes/cylinder.dae" scale="${seg_length/3} ${seg_length/6} ${seg_length/3}" /-->
+        </geometry>
+    </visual>
+    <collision>
+      <origin xyz="${seg_length/2} 0 0" rpy="0 0 0" />
+      <geometry>
+          <mesh filename="package://testbot_description/meshes/cube.dae"
+              scale="${seg_length/3} ${seg_width/2} ${seg_height/2}" />
+        <!--cylinder length="${seg_length/6}" radius="${seg_length/3}" /-->
       </geometry>
     </collision>
     <inertial>
-        <origin xyz="0 0 0" rpy="0 0 0" />
+        <origin xyz="${seg_length/2} 0 0" rpy="0 0 0" />
         <mass value="1" />
         <inertia
@@ -177,11 +200,10 @@
         <child link="head" />
         <origin xyz="0 0 0" rpy="0 0 0" />
-        <axis xyz="0 0 1" />
   </joint>
 <xacro:segment parent="head" postfix="1" length="${seg_length}" width="${seg_width}" height="${seg_height}" />
 <xacro:segment parent="link_1" postfix="2" length="${seg_length}" width="${seg_width}" height="${seg_height}" />
 <xacro:segment parent="link_2" postfix="3" length="${seg_length}" width="${seg_width}" height="${seg_height}" />
+<!--
 <xacro:segment parent="link_3" postfix="4" length="${seg_length}" width="${seg_width}" height="${seg_height}" />
-<!--
 <xacro:segment parent="link_4" postfix="5" length="${seg_length}" width="${seg_width}" height="${seg_height}" />
 <xacro:segment parent="link_5" postfix="6" length="${seg_length}" width="${seg_width}" height="${seg_height}" />

Commit message: I thought placing the projector on the revolutely jointed link would work correctly, but it is still glitchy when the projector is at an angle.  Next create an intermediary revolute joint and attach the projector to that.

File: testbot_description/urdf/testbot.xacro (robot description, xacro)
@@ -201,11 +201,21 @@
         <origin xyz="0 0 0" rpy="0 0 0" />
   </joint>
+<!-- this one doesn't work correctly because it is attached to a fixed link -->
 <gazebo reference="head">
-  <!--sensor type="projector" name="projector_tester"-->
-  <projector name="projector_test1">
-    <pose>0 0 0 0 0 0</pose>
-    <!-- this isn't getting loaded properly -->
-    <!--texture>$(find projector_test)/urdf/test_pattern.png</texture-->
-    <!-- this doesn't work even with setting GAZEBO_RESOURCE_PATH -->
+  <projector name="projector_test_head">
+    <pose>${seg_length/2} 0 0 1.57 0 0</pose>
+    <texture>test_pattern.png</texture>
+    <!--texture>stereo_projection_pattern_high_res_red.png</texture-->
+    <fov>0.95</fov>
+    <near_clip>0.1</near_clip>
+    <far_clip>10.0</far_clip>
+  </projector>
+</gazebo>
+<!-- this works fine because it is attached to a revolute jointed link-->
+<!--link name="link_projector_test_1">
+</link-->
+<gazebo reference="link_1">
+  <projector name="projector_test_1">
+    <pose>${seg_length/2} 0 0 1.57 0 0</pose>
     <texture>test_pattern.png</texture>
     <!--texture>stereo_projection_pattern_high_res_red.png</texture-->

Commit message: Putting another joint in the loop didn't help much (same glitchy results), making the joint fixed as it is here causes the projector to disappear entirely.

File: testbot_description/urdf/testbot.xacro (robot description, xacro)
@@ -212,10 +212,38 @@
   </projector>
 </gazebo>
+<joint name="joint_projector_test_1" type="fixed">
+  <parent link="head" />
+  <child link="link_projector_test_1" />
+  <origin xyz="0 0.23 0" rpy="0 0 0" />
+<!--  <axis xyz="0 1 0" />
+  <limit effort="1000.0" upper="0.0001" lower="-0.0001" velocity="0.5" />
+</joint>
+-->
 <!-- this works fine because it is attached to a revolute jointed link-->
-<!--link name="link_projector_test_1">
-</link-->
-<gazebo reference="link_1">
+<link name="link_projector_test_1">
+    <visual>
+      <origin xyz="0 0 0" rpy="0 0 0" />
+      <geometry>
+        <box size="0.05 0.05 0.05"/>
+      </geometry>
+    </visual>
+    <collision>
+      <origin xyz="0 0 0" rpy="0 0 0" />
+      <geometry>
+        <box size="0.05 0.05 0.05"/>
+      </geometry>
+    </collision>
+    <inertial>
+        <origin xyz="0 0 0" rpy="0 0 0" />
+        <mass value="1" />
+        <inertia
+          ixx="1.0" ixy="0.0" ixz="0.0"
+          iyy="1.0" iyz="0.0"
+          izz="1.0" />
+    </inertial>
+</link>
+<gazebo reference="link_projector_test_1">
   <projector name="projector_test_1">
-    <pose>${seg_length/2} 0 0 1.57 0 0</pose>
+    <pose>0 0 0 1.57 0 0</pose>
     <texture>test_pattern.png</texture>
     <!--texture>stereo_projection_pattern_high_res_red.png</texture-->

Commit message: This arrangment looks to be working, but try a few more orientations.

File: testbot_description/urdf/testbot.xacro (robot description, xacro)
@@ -204,4 +204,5 @@
 <gazebo reference="head">
   <projector name="projector_test_head">
+    <!-- none of the translations or rotations applied here have any effect -->
     <pose>${seg_length/2} 0 0 1.57 0 0</pose>
     <texture>test_pattern.png</texture>
@@ -212,12 +213,12 @@
   </projector>
 </gazebo>
-<joint name="joint_projector_test_1" type="fixed">
+<!-- try putting a projector onto another link -->
+<joint name="joint_projector_test_1" type="revolute">
   <parent link="head" />
   <child link="link_projector_test_1" />
-  <origin xyz="0 0.23 0" rpy="0 0 0" />
-<!--  <axis xyz="0 1 0" />
+  <origin xyz="0 0.23 0" rpy="1.57 0 0" />
+  <axis xyz="0 1 0" />
   <limit effort="1000.0" upper="0.0001" lower="-0.0001" velocity="0.5" />
 </joint>
--->
 <!-- this works fine because it is attached to a revolute jointed link-->
 <link name="link_projector_test_1">
@@ -245,5 +246,5 @@
 <gazebo reference="link_projector_test_1">
   <projector name="projector_test_1">
-    <pose>0 0 0 1.57 0 0</pose>
+    <pose>0 0 0 0 0 0</pose>
     <texture>test_pattern.png</texture>
     <!--texture>stereo_projection_pattern_high_res_red.png</texture-->

Commit message: This orientation looks good too, try flipping to fixed again.

File: testbot_description/urdf/testbot.xacro (robot description, xacro)
@@ -217,5 +217,5 @@
   <parent link="head" />
   <child link="link_projector_test_1" />
-  <origin xyz="0 0.23 0" rpy="1.57 0 0" />
+  <origin xyz="0 0.23 0" rpy="0 1.57 0" />
   <axis xyz="0 1 0" />
   <limit effort="1000.0" upper="0.0001" lower="-0.0001" velocity="0.5" />

Commit message: Fixed makes the texture disappear

File: testbot_description/urdf/testbot.xacro (robot description, xacro)
@@ -214,10 +214,12 @@
 </gazebo>
 <!-- try putting a projector onto another link -->
-<joint name="joint_projector_test_1" type="revolute">
+<joint name="joint_projector_test_1" type="fixed">
   <parent link="head" />
   <child link="link_projector_test_1" />
   <origin xyz="0 0.23 0" rpy="0 1.57 0" />
+<!--
   <axis xyz="0 1 0" />
   <limit effort="1000.0" upper="0.0001" lower="-0.0001" velocity="0.5" />
+-->
 </joint>
 <!-- this works fine because it is attached to a revolute jointed link-->

Commit message: Showing the pose setting not working again.

File: testbot_description/urdf/testbot.xacro (robot description, xacro)
@@ -214,12 +214,10 @@
 </gazebo>
 <!-- try putting a projector onto another link -->
-<joint name="joint_projector_test_1" type="fixed">
+<joint name="joint_projector_test_1" type="revolute">
   <parent link="head" />
   <child link="link_projector_test_1" />
-  <origin xyz="0 0.23 0" rpy="0 1.57 0" />
-<!--
+  <origin xyz="0 0.23 0" rpy="0 0 0" />
   <axis xyz="0 1 0" />
   <limit effort="1000.0" upper="0.0001" lower="-0.0001" velocity="0.5" />
--->
 </joint>
 <!-- this works fine because it is attached to a revolute jointed link-->
@@ -248,5 +246,6 @@
 <gazebo reference="link_projector_test_1">
   <projector name="projector_test_1">
-    <pose>0 0 0 0 0 0</pose>
+    <!-- setting the pose will produce glitches even when attached to a revolute joint -->
+    <pose>0 0 0 0 1.57 0</pose>
     <texture>test_pattern.png</texture>
     <!--texture>stereo_projection_pattern_high_res_red.png</texture-->
