Commit message: It looks like rospy tf isn't listening to tf_static at all

File: tf_test/urdf/tf_test.xacro (robot description, xacro)
@@ -3,11 +3,18 @@
 <link name="map">
 </link>
+<link name="link1">
+</link>
+<joint name="joint1" type="fixed">
+  <parent link="map"/>
+  <child link="link1"/>
+  <origin xyz="0 0 0" rpy="0 0 0"/>
+</joint>
 <link name="test_link">
 </link>
 <joint name="test_joint" type="revolute">
-  <parent link="map"/>
+  <parent link="link1"/>
   <child link="test_link"/>
   <origin xyz="0 0 0" rpy="0 0 0"/>
-  <axis xyz="0 0 1" />
+  <axis xyz="0 0 1"/>
   <limit effort="5000" lower="-0.5" upper="0.5" velocity="50"/>
 </joint>

Commit message: Finally figured out that rospy tf is broken in jade, need to use tf2 https://github.com/ros/geometry/issues/117

File: tf_test/urdf/tf_test.xacro (robot description, xacro)
@@ -6,7 +6,16 @@
 </link>
 <joint name="joint1" type="fixed">
-  <parent link="map"/>
+  <parent link="link2"/>
   <child link="link1"/>
   <origin xyz="0 0 0" rpy="0 0 0"/>
+</joint>
+<link name="link2">
+</link>
+<joint name="joint2" type="revolute">
+  <parent link="map"/>
+  <child link="link2"/>
+  <origin xyz="0 0 0" rpy="0 0 0"/>
+  <axis xyz="0 0 1"/>
+  <limit effort="5000" lower="-0.5" upper="0.5" velocity="50"/>
 </joint>
 <link name="test_link">
